File: stm32_rf_usb_logger/stm32_rf_usb_logger.kicad_sch (KiCad schematic)
At the start: 39 parts, among them J1 SWD, J2 USB_B_Micro, J3 Conn_Coaxial, J4 RFShield_OnePiece, U1 XC6206PxxxMR, U2 STM32L432KBUx, U3 USBLC6-2SC6, U4 nRF24L01P, Y2 16MHz

Commit message: completed layout
Parts:
- J4: footprint (none) -> RF_Shielding:Laird_Technologies_BMI-S-102_16.50x16.50mm
- renumbered C2 to C1, C14 to C12, C16 to C13, C15 to C14, C7 to C15, C12 to C16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
Connections:
- net GND: now also J4.1 (Shield)
